File: Hardware/LoRa-Monitor/PowerSupply.kicad_sch (KiCad schematic)
At the start: 41 parts, among them U1 IRM-05-5, U11 TPS63021DSJR, U12 NXE1S0303MC, U13 NXE1S0303MC, U9 BQ24072RGT

Commit message: Finished routing and DRC gives 0 errors.
Parts:
- L2, L3: footprint DeviceComponents:L_0806_2016Metric -> Inductor_SMD:L_1210_3225Metric_Pad1.42x2.65mm_HandSolder
Changed lines of the file:
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@@
 			)
 		)
-		(property "Footprint" "DeviceComponents:L_0806_2016Metric"
+		(property "Footprint" "Inductor_SMD:L_1210_3225Metric_Pad1.42x2.65mm_HandSolder"
 			(at 232.41 110.49 0)
 			(hide yes)
@@
 			)
 		)
-		(property "Footprint" "DeviceComponents:L_0806_2016Metric"
+		(property "Footprint" "Inductor_SMD:L_1210_3225Metric_Pad1.42x2.65mm_HandSolder"
 			(at 232.41 139.7 0)
 			(hide yes)

Commit message: Added parameters for the productions files, changed components on LCSC to reduce the price of BoM, minimal changes on the routing.
Parts:
- C10, C11: LCSC Part # (none) -> C28323
- C12: value 4.7uF 50V X7R -> 4.7uF 25V X7R; LCSC Part # (none) -> C1779
- C13, C8: LCSC Part # (none) -> C7223
- C14, C15: LCSC Part # (none) -> C15850
- C16, C19, C20: LCSC Part # (none) -> C45783
- C17, C21: value 100nF -> 100nF 50V X7R; LCSC Part # (none) -> C49678
- C18, C22: value 1uF -> 1uF 50V X7R; LCSC Part # (none) -> C28323
- C9: LCSC Part # (none) -> C49678
- D5: LCSC Part # (none) -> C84256
- F1: LCSC Part # (none) -> C83797
- L1: LCSC Part # (none) -> C161082
- L2, L3: LCSC Part # (none) -> C250232
- R103: LCSC Part # (none) -> C483162
- R104, R107, R110, R19, R31, R32: LCSC Part # (none) -> C17414
- R105, R108, R109, R33: LCSC Part # (none) -> C185294
- R106: LCSC Part # (none) -> C17460
- R34: LCSC Part # (none) -> C55566
- RV1: LCSC Part # (none) -> C2656193
- U1: LCSC Part # (none) -> C48603696
- U11: FT Rotation Offset (none) -> -90; LCSC Part # (none) -> C202140
- U12, U13: FT Position Offset (none) -> 0,1.27; FT Rotation Offset (none) -> -90; LCSC Part # (none) -> C20606969
- U9: LCSC Part # (none) -> C140288
