File: Hardware/LoRa-Monitor/PowerSupply.kicad_sch (KiCad schematic)
At the start: 41 parts, among them U1 IRM-05-5, U11 TPS63021DSJR, U12 NXE1S0303MC, U13 NXE1S0303MC, U9 BQ24072RGT

Commit message: Changed the RS485-TTL translator and its relevent componentes (Power source and optocuplers) for a simpler and easier solution using the ADM2582.
Parts:
- removed C14: 10uF, Capacitor_SMD:C_0805_2012Metric, symbol Device:C
- removed C18: 1uF 50V X7R, Capacitor_SMD:C_0805_2012Metric, symbol Device:C
- removed L2: 15uH, Inductor_SMD:L_1210_3225Metric_Pad1.42x2.65mm_HandSolder, symbol Device:L
- removed U12: NXE1S0303MC, Converter_DCDC:Converter_DCDC_Murata_NXExSxxxxMC_SMD, symbol Regulator_Switching:NXE1S0303MC
- renumbered C13 to C18, C16 to C19, C17 to C20, C8 to C22, C9 to C23, C19 to C24, C20 to C25, C10 to C26, C22 to C27, C12 to C28, C11 to C29, C15 to C30, D5 to D6, L3 to L2, R110 to R45, R32 to R46, R19 to R47, R103 to R48, R31 to R49, R104 to R50, R33 to R51, R34 to R52, R108 to R53, R109 to R54, R107 to R55, R105 to R56, R106 to R57, U1 to U6, U11 to U7, U9 to U8, U13 to U9
Other:
- moved on the sheet: C27, C30, L2, U9
