File: Hardware/LoRa-Monitor/Connectors.kicad_sch (KiCad schematic)
At the start: 13 parts, among them J1 USB_C_Receptacle_USB2.0_16P, J10 AudioJack3, J11 Screw_Terminal_01x02, J12 Screw_Terminal_01x02, J13 Conn_01x02_Pin, J14 Conn_01x02_Pin, J3 Conn_02x03_Odd_Even, J4 Conn_Coaxial, J5 Screw_Terminal_01x02, J6 Screw_Terminal_01x02, J7 AudioJack3, J8 AudioJack3, J9 Screw_Terminal_01x04

Commit message: Finished routing and DRC gives 0 errors.
Parts:
- removed J5: Screw_Terminal_01x02, TerminalBlock_Phoenix:TerminalBlock_Phoenix_PT-1,5-2-5.0-H_1x02_P5.00mm_Horizontal, symbol Connector:Screw_Terminal_01x02
- added H1, H2, H3, H4, H5, H6: MountingHole, MountingHole:MountingHole_3.2mm_M3_DIN965, symbol Mechanical:MountingHole
- added J15: Screw_Terminal_01x03, TerminalBlock_Phoenix:TerminalBlock_Phoenix_PT-1,5-3-5.0-H_1x03_P5.00mm_Horizontal, symbol Connector:Screw_Terminal_01x03
- J4: footprint Connector_Coaxial:SMA_Amphenol_901-144_Vertical -> Connector_Coaxial:U.FL_Molex_MCRF_73412-0110_Vertical
Connections:
- net 485_A: now also J15.1 (Pin_1)
- net 485_B: now also J15.2 (Pin_2)
- new net GND_485: J15.3 (Pin_3)

Commit message: Added parameters for the productions files, changed components on LCSC to reduce the price of BoM, minimal changes on the routing.
Parts:
- J1: FT Position Offset (none) -> 0,1.4605; LCSC Part # (none) -> C165948
- J10, J7, J8: FT Position Offset (none) -> 0,1.0795; FT Rotation Offset (none) -> 180; LCSC Part # (none) -> C20182914
- J11, J12, J6: LCSC Part # (none) -> C3819953
- J13, J14: FT Rotation Offset (none) -> 180; LCSC Part # (none) -> C131337
- J15: LCSC Part # (none) -> C3816891
- J4: LCSC Part # (none) -> C434806
- J9: LCSC Part # (none) -> C3817931

Commit message: Changed the RS485-TTL translator and its relevent componentes (Power source and optocuplers) for a simpler and easier solution using the ADM2582.
Parts:
- renumbered J11 to J10, J12 to J11, J7 to J12, J8 to J13, J10 to J14, J3 to J2, J1 to J3, J13 to J5, J14 to J6, J9 to J7, J15 to J8, J6 to J9
Changed lines of the file:
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@@
 		(in_pos_files yes)
 		(dnp no)
-		(property "Reference" "#PWR0134"
+		(property "Reference" "#PWR050"
 			(at 102.87 130.81 0)
 			(hide yes)
@@
 			(project "LoRa-Monitor"
 				(path "/7510cc7d-c141-46d4-8947-7def3af8cf35/b9106b62-0c4d-45f8-8fff-77bde9d1c249"
-					(reference "#PWR0134")
+					(reference "#PWR050")
 					(unit 1)
 				)
@@
 		(in_pos_files yes)
 		(dnp no)
-		(property "Reference" "#PWR0135"
+		(property "Reference" "#PWR052"
 			(at 154.94 186.69 0)
 			(hide yes)
@@
 			(project "LoRa-Monitor"
 				(path "/7510cc7d-c141-46d4-8947-7def3af8cf35/b9106b62-0c4d-45f8-8fff-77bde9d1c249"
-					(reference "#PWR0135")
+					(reference "#PWR052")
 					(unit 1)
 				)
@@
 		(dnp no)
 		(fields_autoplaced yes)
-		(property "Reference" "J11"
+		(property "Reference" "J10"
 			(at 238.76 69.8499 0)
 			(show_name no)
@@
 			(project "LoRa-Monitor"
 				(path "/7510cc7d-c141-46d4-8947-7def3af8cf35/b9106b62-0c4d-45f8-8fff-77bde9d1c249"
-					(reference "J11")
+					(reference "J10")
 					(unit 1)
 				)
@@
 		(dnp no)
 		(fields_autoplaced yes)
-		(property "Reference" "J13"
+		(property "Reference" "J5"
 			(at 174.625 134.62 0)
 			(show_name no)
@@
 			(project "LoRa-Monitor"
 				(path "/7510cc7d-c141-46d4-8947-7def3af8cf35/b9106b62-0c4d-45f8-8fff-77bde9d1c249"
-					(reference "J13")
+					(reference "J5")
 					(unit 1)
 				)
@@
 		(in_pos_files yes)
 		(dnp no)
-		(property "Reference" "J8"
+		(property "Reference" "J13"
 			(at 238.125 109.22 0)
 			(show_name no)
@@
 			(project "LoRa-Monitor"
 				(path "/7510cc7d-c141-46d4-8947-7def3af8cf35/b9106b62-0c4d-45f8-8fff-77bde9d1c249"
-					(reference "J8")
+					(reference "J13")
 					(unit 1)
 				)
@@
 		(dnp no)
 		(fields_autoplaced yes)
-		(property "Reference" "J9"
+		(property "Reference" "J7"
 			(at 238.76 31.7499 0)
 			(show_name no)
@@
 			(project "LoRa-Monitor"
 				(path "/7510cc7d-c141-46d4-8947-7def3af8cf35/b9106b62-0c4d-45f8-8fff-77bde9d1c249"
-					(reference "J9")
+					(reference "J7")
 					(unit 1)
 				)
@@
 		(dnp no)
 		(fields_autoplaced yes)
-		(property "Reference" "J6"
+		(property "Reference" "J9"
 			(at 238.76 59.6899 0)
 			(show_name no)
@@
 			(project "LoRa-Monitor"
 				(path "/7510cc7d-c141-46d4-8947-7def3af8cf35/b9106b62-0c4d-45f8-8fff-77bde9d1c249"
-					(reference "J6")
+					(reference "J9")
 					(unit 1)
 				)
@@
 		(dnp no)
 		(fields_autoplaced yes)
-		(property "Reference" "#PWR078"
+		(property "Reference" "#PWR051"
 			(at 130.81 194.31 0)
 			(hide yes)
@@
 			(project "LoRa-Monitor"
 				(path "/7510cc7d-c141-46d4-8947-7def3af8cf35/b9106b62-0c4d-45f8-8fff-77bde9d1c249"
-					(reference "#PWR078")
+					(reference "#PWR051")
 					(unit 1)
 				)
@@
 		(in_pos_files yes)
 		(dnp no)
-		(property "Reference" "#PWR0136"
+		(property "Reference" "#PWR053"
 			(at 154.94 194.31 0)
 			(hide yes)
@@
 			(project "LoRa-Monitor"
 				(path "/7510cc7d-c141-46d4-8947-7def3af8cf35/b9106b62-0c4d-45f8-8fff-77bde9d1c249"
-					(reference "#PWR0136")
+					(reference "#PWR053")
 					(unit 1)
 				)
@@
 		(dnp no)
 		(fields_autoplaced yes)
-		(property "Reference" "J14"
+		(property "Reference" "J6"
 			(at 174.625 144.78 0)
 			(show_name no)
@@
 			(project "LoRa-Monitor"
 				(path "/7510cc7d-c141-46d4-8947-7def3af8cf35/b9106b62-0c4d-45f8-8fff-77bde9d1c249"
-					(reference "J14")
+					(reference "J6")
 					(unit 1)
 				)
@@
 		(in_pos_files yes)
 		(dnp no)
-		(property "Reference" "J7"
+		(property "Reference" "J12"
 			(at 238.125 93.98 0)
 			(show_name no)
@@
 			(project "LoRa-Monitor"
 				(path "/7510cc7d-c141-46d4-8947-7def3af8cf35/b9106b62-0c4d-45f8-8fff-77bde9d1c249"
-					(reference "J7")
+					(reference "J12")
 					(unit 1)
 				)
@@
 		(in_pos_files yes)
 		(dnp no)
-		(property "Reference" "#PWR0137"
+		(property "Reference" "#PWR047"
 			(at 64.77 46.99 0)
 			(hide yes)
@@
 			(project "LoRa-Monitor"
 				(path "/7510cc7d-c141-46d4-8947-7def3af8cf35/b9106b62-0c4d-45f8-8fff-77bde9d1c249"
-					(reference "#PWR0137")
+					(reference "#PWR047")
 					(unit 1)
 				)
@@
 		(dnp no)
 		(fields_autoplaced yes)
-		(property "Reference" "J15"
+		(property "Reference" "J8"
 			(at 238.76 44.4499 0)
 			(show_name no)
@@
 			(project "LoRa-Monitor"
 				(path "/7510cc7d-c141-46d4-8947-7def3af8cf35/b9106b62-0c4d-45f8-8fff-77bde9d1c249"
-					(reference "J15")
+					(reference "J8")
 					(unit 1)
 				)
@@
 		(dnp no)
 		(fields_autoplaced yes)
-		(property "Reference" "J1"
+		(property "Reference" "J3"
 			(at 96.52 26.67 0)
 			(show_name no)
@@
 			(project "LoRa-Monitor"
 				(path "/7510cc7d-c141-46d4-8947-7def3af8cf35/b9106b62-0c4d-45f8-8fff-77bde9d1c249"
-					(reference "J1")
+					(reference "J3")
 					(unit 1)
 				)
@@
 		(dnp no)
 		(fields_autoplaced yes)
-		(property "Reference" "J12"
+		(property "Reference" "J11"
 			(at 238.76 78.7399 0)
 			(show_name no)
@@
 			(project "LoRa-Monitor"
 				(path "/7510cc7d-c141-46d4-8947-7def3af8cf35/b9106b62-0c4d-45f8-8fff-77bde9d1c249"
-					(reference "J12")
+					(reference "J11")
 					(unit 1)
 				)
@@
 		(dnp no)
 		(fields_autoplaced yes)
-		(property "Reference" "#PWR0144"
+		(property "Reference" "#PWR054"
 			(at 229.87 55.88 0)
 			(hide yes)
@@
 			(project "LoRa-Monitor"
 				(path "/7510cc7d-c141-46d4-8947-7def3af8cf35/b9106b62-0c4d-45f8-8fff-77bde9d1c249"
-					(reference "#PWR0144")
+					(reference "#PWR054")
 					(unit 1)
 				)
@@
 		(in_pos_files yes)
 		(dnp no)
-		(property "Reference" "J10"
+		(property "Reference" "J14"
 			(at 238.125 124.46 0)
 			(show_name no)
@@
 			(project "LoRa-Monitor"
 				(path "/7510cc7d-c141-46d4-8947-7def3af8cf35/b9106b62-0c4d-45f8-8fff-77bde9d1c249"
-					(reference "J10")
+					(reference "J14")
 					(unit 1)
 				)
@@
 		(in_pos_files yes)
 		(dnp no)
-		(property "Reference" "#PWR0138"
+		(property "Reference" "#PWR048"
 			(at 64.77 59.69 0)
 			(hide yes)
@@
 			(project "LoRa-Monitor"
 				(path "/7510cc7d-c141-46d4-8947-7def3af8cf35/b9106b62-0c4d-45f8-8fff-77bde9d1c249"
-					(reference "#PWR0138")
+					(reference "#PWR048")
 					(unit 1)
 				)
@@
 		(in_pos_files yes)
 		(dnp no)
-		(property "Reference" "#PWR0133"
+		(property "Reference" "#PWR049"
 			(at 96.52 81.28 0)
 			(hide yes)
@@
 			(project "LoRa-Monitor"
 				(path "/7510cc7d-c141-46d4-8947-7def3af8cf35/b9106b62-0c4d-45f8-8fff-77bde9d1c249"
-					(reference "#PWR0133")
+					(reference "#PWR049")
 					(unit 1)
 				)
@@
 		(dnp no)
 		(fields_autoplaced yes)
-		(property "Reference" "J3"
+		(property "Reference" "J2"
 			(at 55.88 39.37 0)
 			(show_name no)
@@
 			(project "LoRa-Monitor"
 				(path "/7510cc7d-c141-46d4-8947-7def3af8cf35/b9106b62-0c4d-45f8-8fff-77bde9d1c249"
-					(reference "J3")
+					(reference "J2")
 					(unit 1)
 				)
