File: Hardware/LoRa-Monitor/LoRa-Monitor.kicad_pcb (KiCad board)
At the start: 2 copper layers, 1.4 x 13 mm, 222 parts, among them J1 USB_C_Receptacle_USB2.0_16P, J10 AudioJack3, J11 Screw_Terminal_01x02, J12 Screw_Terminal_01x02, J13 Conn_01x02_Pin, J14 Conn_01x02_Pin, J2 Micro_SD_Card, J3 Conn_02x03_Odd_Even, J4 Conn_Coaxial, J5 Screw_Terminal_01x02, J6 Screw_Terminal_01x02, J7 AudioJack3, J8 AudioJack3, J9 Screw_Terminal_01x04, Q1 ZXTN25100DFH, Q2 ZXTN25100DFH, Q3 ZXTN25100DFH, Q4 ZXTN25100DFH, Q5 ZXTN25100DFH, Q6 ZXTN25100DFH, U1 IRM-05-5, U10 ESP32-S3-WROOM-1, U11 TPS63021DSJR, U12 NXE1S0303MC, U13 NXE1S0303MC, U14 ATM90E32AS-AU-R, U15 E22-900M30S, U16 ADuM1401xRW, U17 ADuM1401xRW, U18 ADuM1401xRW, U2 ACPL-M61L, U3 ACPL-M61L, U4 ACPL-M61L, U5 ACPL-M61L, U6 ACPL-M61L, U7 ACPL-M61L, U8 MAX3483, U9 BQ24072RGT

Commit message: Finished the first component disposition
Parts:
- R114, R49, R50, R51, R52, R53, R54, R57, R58, R59, R60, R61, R62, R63, R66, R67, R68, R69, R70, R71, R72: footprint Resistor_SMD:R_0805_2012Metric -> Resistor_SMD:R_1206_3216Metric
- moved C33 562.8 mm to (67.9, 109.5)
- moved R65 562.7 mm to (67.9, 111.5)
- moved C32 561.3 mm to (67.9, 113.5)
- moved R64 561.3 mm to (67.9, 115.6)
- moved C24 560.7 mm to (56.8, 107.8), turned to -90 degrees
- moved C26 560.0 mm to (63.6, 90.2), turned to 180 degrees
- moved R112 559.1 mm to (73.3, 86.1), turned to -90 degrees
- moved C25 559.0 mm to (63.6, 92.3), turned to 180 degrees
- moved R113 558.8 mm to (73.3, 89.5), turned to 90 degrees
- moved R111 558.5 mm to (73.3, 92.9), turned to -90 degrees
- moved R44 558.1 mm to (73.3, 96.2), turned to 90 degrees
- moved C23 558.1 mm to (58.9, 107.8), turned to -90 degrees
- moved R87 557.8 mm to (73.3, 99.6), turned to -90 degrees
- moved C29 557.8 mm to (60.1, 92.3)
- moved U14 557.7 mm to (64.3, 99.2)
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Connections:
- J9 pad 1: /Connectors/Uc -> /Connectors/Ua
- J9 pad 3: /Connectors/Ua -> /Connectors/Uc
- R1 pad 1: /Energy meter/IRQ0 -> /Energy meter/ZX0
- R10 pad 1: /Energy Meter Interface Module/PULSE_IN2_3V3 -> /Energy Meter Interface Module/TXD_485
- R11 pad 1: /Energy Meter Interface Module/PULSE_IN3_3V3 -> /Energy Meter Interface Module/EN_485
- R12 pad 1: /LoRa Module/~{RST_E22} -> /Energy Meter Interface Module/RXD_485
- R13 pad 1: /Energy meter/CS_ATM90 -> /Energy Meter Interface Module/PULSE_IN1_3V3
- R14 pad 1: /Energy meter/SCKL_SPI0 -> /Energy Meter Interface Module/PULSE_IN2_3V3
- R15 pad 1: /Energy meter/SDI_SPI0 -> /LoRa Module/~{RST_E22}
- R16 pad 1: /Energy meter/SDO_SPI0 -> /LoRa Module/BUSY_E22
- R17 pad 2: /Energy Meter Interface Module/RXD_485 -> /LoRa Module/DIO1_E22
- R18 pad 2: /Energy Meter Interface Module/TXD_485 -> /MCU/CS_SD
- R2 pad 1: /Energy meter/IRQ1 -> /Energy meter/ZX1
- R21 pad 2: /Energy Meter Interface Module/EN_485 -> /Energy Meter Interface Module/PULSE_IN3_3V3
- R3 pad 1: /Energy meter/WARNOUT -> /MCU/SCLK_SPI1
- R35 pad 2: /LoRa Module/BUSY_E22 -> /Energy meter/SCKL_SPI0
- R36 pad 2: /LoRa Module/DIO1_E22 -> /Energy meter/CS_ATM90
- R37 pad 2: /LoRa Module/DIO2_E22 -> /Energy meter/PM1
- R38 pad 2: /MCU/SDO_SPI1 -> /Energy meter/PM0
- R39 pad 2: /MCU/SDI_SPI1 -> /Energy meter/IRQ1
- R4 pad 1: /Energy meter/PM0 -> /LoRa Module/RXEN_E22
- R40 pad 2: /MCU/SCLK_SPI1 -> /Energy meter/IRQ0
- R41 pad 2: /LoRa Module/CS_E22 -> /Energy meter/WARNOUT
- R42 pad 2: /MCU/CS_SD -> /Energy meter/ZX2
- R47 pad 2: /LoRa Module/RXEN_E22 -> /Energy meter/SDO_SPI0
- R48 pad 2: /LoRa Module/TXEN_E22 -> /Energy meter/SDI_SPI0
- R5 pad 1: /Energy meter/PM1 -> /LoRa Module/TXEN_E22
- R6 pad 1: /Energy meter/ZX0 -> /LoRa Module/DIO2_E22
- R7 pad 1: /Energy meter/ZX1 -> /LoRa Module/CS_E22
- R8 pad 1: /Energy meter/ZX2 -> /MCU/SDO_SPI1
- R9 pad 1: /Energy Meter Interface Module/PULSE_IN1_3V3 -> /MCU/SDI_SPI1
- U17 pad 11: /Energy meter/PM0 -> /Energy meter/ZX0
- U17 pad 12: /Energy meter/ZX2 -> /Energy meter/ZX1
- U17 pad 13: /Energy meter/ZX1 -> /Energy meter/ZX2
- U17 pad 14: /Energy meter/ZX0 -> /Energy meter/WARNOUT
- U17 pad 3: /Energy meter/ZX0_M90 -> /Energy meter/WARNOUT_M90
- U17 pad 4: /Energy meter/ZX1_M90 -> /Energy meter/ZX2_M90
- U17 pad 5: /Energy meter/ZX2_M90 -> /Energy meter/ZX1_M90
- U17 pad 6: /Energy meter/PM0_M90 -> /Energy meter/ZX0_M90
- U18 pad 11: /Energy meter/PM1 -> /Energy meter/IRQ0
- U18 pad 12: /Energy meter/WARNOUT -> /Energy meter/IRQ1
- U18 pad 13: /Energy meter/IRQ1 -> /Energy meter/PM0
- U18 pad 14: /Energy meter/IRQ0 -> /Energy meter/PM1
- U18 pad 3: /Energy meter/IRQ0_M90 -> /Energy meter/PM1_M90
- U18 pad 4: /Energy meter/IRQ1_M90 -> /Energy meter/PM0_M90
- U18 pad 5: /Energy meter/WARNOUT_M90 -> /Energy meter/IRQ1_M90
- U18 pad 6: /Energy meter/PM1_M90 -> /Energy meter/IRQ0_M90
Routing:
- net /Connectors/USB_D+: track 27.5 -> 0.00 mm
- net /Connectors/USB_D-: track 26.7 -> 0.00 mm
- net (no net): track 14.9 -> 0.00 mm
