File: Hardware/LoRa-Monitor/EnergyMeter.kicad_sch (KiCad schematic)
At the start: 88 parts, among them U14 ATM90E32AS-AU-R, U16 ADuM1401xRW, U17 ADuM1401xRW, U18 ADuM1401xRW, Y1 16.384MHz

Commit message: Changed the RS485-TTL translator and its relevent componentes (Power source and optocuplers) for a simpler and easier solution using the ADM2582.
Parts:
- renumbered C36 to C31, C37 to C32, C38 to C33, C39 to C34, C40 to C35, C41 to C36, C30 to C37, C32 to C38, C34 to C39, C52 to C40, C31 to C41, C33 to C42, C35 to C43, C53 to C44, C54 to C45, C27 to C46, C55 to C47, C56 to C48, C23 to C49, C28 to C50, C24 to C51, C25 to C52, C29 to C53, C57 to C54, C26 to C55, R91 to R100, R56 to R101, R65 to R102, R74 to R103, R94 to R104, R113 to R105, R112 to R106, R111 to R107, R92 to R108, R44 to R109, R43 to R110, R87 to R111, R88 to R112, R93 to R113, R90 to R114, R89 to R115, R114 to R58, R57 to R59, R66 to R60, R49 to R61, R58 to R62, R67 to R63, R50 to R64, R59 to R65, R68 to R66, R116 to R67, R117 to R68, R118 to R69, R119 to R70, R120 to R71, R121 to R72, R75 to R73, R76 to R74, R79 to R75, R80 to R76, R83 to R77, R84 to R78, R51 to R79, R60 to R80, R69 to R81, R77 to R82, R78 to R83, R81 to R84, R82 to R85, R85 to R86, R86 to R87, R52 to R88, R61 to R89, R70 to R90, R53 to R91, R62 to R92, R71 to R93, R54 to R94, R63 to R95, R72 to R96, R55 to R97, R64 to R98, R73 to R99, U18 to U10, U17 to U11, U14 to U12, U16 to U13
