File: Hardware/LoRa-Monitor/Interfaces.kicad_sch (KiCad schematic)
At the start: 37 parts, among them Q1 ZXTN25100DFH, Q2 ZXTN25100DFH, Q3 ZXTN25100DFH, Q4 ZXTN25100DFH, Q5 ZXTN25100DFH, Q6 ZXTN25100DFH, U2 ACPL-M61L, U3 ACPL-M61L, U4 ACPL-M61L, U5 ACPL-M61L, U6 ACPL-M61L, U7 ACPL-M61L, U8 MAX3483

Commit message: Added parameters for the productions files, changed components on LCSC to reduce the price of BoM, minimal changes on the routing.
Parts:
- removed Q1, Q2, Q3, Q4, Q5, Q6: ZXTN25100DFH, Package_TO_SOT_SMD:SOT-23, symbol Transistor_BJT:Q_NPN_BEC
- removed U8: MAX3483, Package_SO:SOIC-8_3.9x4.9mm_P1.27mm, symbol Interface_UART:MAX3483
- added Q1, Q2, Q3, Q4, Q5, Q6: MMBT5551L, Package_TO_SOT_SMD:SOT-23, symbol Transistor_BJT:MMBT5551L
- added U8: MAX3485, Package_SO:SOIC-8_3.9x4.9mm_P1.27mm, symbol Interface_UART:MAX3485
- C1, C2, C3, C4, C5, C6, C7: value 0.1 uF -> 100nF 50V X7R; LCSC Part # (none) -> C49678
- D1, D2, D3: LCSC Part # (none) -> C113963
- D4: LCSC Part # (none) -> C521963
- R102, R20, R22: LCSC Part # (none) -> C17902
- R23, R24, R25: LCSC Part # (none) -> C17408
- R26, R27, R28: LCSC Part # (none) -> C17630
- R29, R30: LCSC Part # (none) -> C17414
- R_TERM1: LCSC Part # (none) -> C17437
- U2, U3, U4, U5, U6, U7: FT Rotation Offset (none) -> -90; LCSC Part # (none) -> C691956
Connections:
- net +3.3V_485: now also U8.8 (VCC)
- net 485_A: now also U8.6 (A)
- net 485_B: now also U8.7 (B)
- net GND_485: now also U8.5 (GND)
- net PULSE_IN1-: now also Q1.2 (E)
- net PULSE_IN2-: now also Q2.2 (E)
- net PULSE_IN3-: now also Q3.2 (E)
- net at R24.1: now also Q2.1 (B), Q5.2 (E)
- net at R20.2: now also Q1.3 (C), Q4.1 (B)
- net at R23.1: now also Q1.1 (B), Q4.2 (E)
- net at R102.2: now also Q2.3 (C), Q5.1 (B)
- net at U3.3 (C): now also Q5.3 (C)
- net at U4.3 (C): now also Q6.3 (C)
- net at R28.2: now also U8.1 (RO)
- net at U6.5 (VO): now also U8.2 (~{RE}), U8.3 (DE)
- net at U7.5 (VO): now also U8.4 (DI)
- net at R22.2: now also Q3.3 (C), Q6.1 (B)
- net at R25.1: now also Q3.1 (B), Q6.2 (E)
- net at U2.3 (C): now also Q4.3 (C)

Commit message: Changed the RS485-TTL translator and its relevent componentes (Power source and optocuplers) for a simpler and easier solution using the ADM2582.
Parts:
- removed C4, C6, C7: 100nF 50V X7R, Capacitor_SMD:C_0805_2012Metric, symbol Device:C
- removed R26, R27, R28: 330R, Resistor_SMD:R_0805_2012Metric, symbol Device:R
- removed U5, U6, U7: ACPL-M61L, DeviceComponents:SO-5_4.39x3.84mm_P1.27mm, symbol DeviceComponents:ACPL-M61L
- removed U8: MAX3485, Package_SO:SOIC-8_3.9x4.9mm_P1.27mm, symbol Interface_UART:MAX3485
- added C10, C11, C16: 100nF, Capacitor_SMD:C_0805_2012Metric, symbol Device:C
- added C12, C15: 10uF, Capacitor_SMD:C_0805_2012Metric, symbol Device:C
- added C13, C17: 10nF, Capacitor_SMD:C_0805_2012Metric, symbol Device:C
- added FB1, FB2: FerriteBead, Inductor_SMD:L_0603_1608Metric, symbol Device:FerriteBead
- added U5: ADM2582E, Package_SO:SOIC-20W_7.5x12.8mm_P1.27mm, symbol Interface_UART:ADM2582E
- C14: renamed from C5; value 100nF 50V X7R -> 100nF
- renumbered C1 to C7, C2 to C8, C3 to C9, D1 to D2, D2 to D3, D3 to D4, D4 to D5, R20 to R37, R102 to R38, R22 to R39, R23 to R40, R24 to R41, R25 to R42, R29 to R43, R30 to R44
Connections:
- net +3.3V: now also C10.1, C11.1, C12.1, C13.1, U5.2 (VCC), U5.8 (VCC)
- net +3.3V_485: now also C15.1, C16.1, C17.1, FB1.2, U5.19 (Visoin); no longer C14.1
- net 485_A: now also U5.13 (Y), U5.18 (A)
- net 485_B: now also U5.15 (Z), U5.17 (B)
- net EN_485: now also U5.5 (~{RE}), U5.6 (DE)
- net GND: now also C10.2, C11.2, C12.2, C13.2, U5.1 (GND1), U5.10 (GND1), U5.3 (GND1), U5.9 (GND1)
- net GND_485: now also C15.2, C16.2, C17.2, FB2.2, U5.16 (GND2), U5.20 (GND2); no longer C14.2
- net RXD_485: now also U5.4 (RxD)
- net TXD_485: now also U5.7 (TxD)
- new net: C14.2, FB2.1, U5.11 (GND2), U5.14 (GND2)
- new net: C14.1, FB1.1, U5.12 (Visoout)
Other:
- moved on the sheet: C14, D5, JP1, R43, R44, R_TERM1
