File: Hardware/LoRa-Monitor/LoRaModule.kicad_sch (KiCad schematic)
At the start: 10 parts, among them U15 E22-900M30S

Commit message: Added parameters for the productions files, changed components on LCSC to reduce the price of BoM, minimal changes on the routing.
Parts:
- C42, C49: value 100nF -> 100nF 50V X7R; LCSC Part # (none) -> C49678
- C48, C50, C51: LCSC Part # (none) -> C15850
- R100, R95, R98, R99: LCSC Part # (none) -> C17414
- U15: FT Position Offset (none) -> 0,1.397; LCSC Part # (none) -> C411294

Commit message: Changed the RS485-TTL translator and its relevent componentes (Power source and optocuplers) for a simpler and easier solution using the ADM2582.
Parts:
- renumbered C42 to C56, C50 to C57, C51 to C58, C48 to C59, C49 to C60, R98 to R116, R95 to R117, R99 to R118, R100 to R119, U15 to U14
Changed lines of the file:
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@@
 		(dnp no)
 		(fields_autoplaced yes)
-		(property "Reference" "C42"
+		(property "Reference" "C56"
 			(at 97.79 77.4699 0)
 			(show_name no)
@@
 			(project "LoRa-Monitor"
 				(path "/7510cc7d-c141-46d4-8947-7def3af8cf35/004b7f1f-ea7b-4526-8ebc-4e4b164bf3f3"
-					(reference "C42")
+					(reference "C56")
 					(unit 1)
 				)
@@
 		(in_pos_files yes)
 		(dnp no)
-		(property "Reference" "#PWR0130"
+		(property "Reference" "#PWR0129"
 			(at 128.27 135.89 0)
 			(hide yes)
@@
 			(project "LoRa-Monitor"
 				(path "/7510cc7d-c141-46d4-8947-7def3af8cf35/004b7f1f-ea7b-4526-8ebc-4e4b164bf3f3"
-					(reference "#PWR0130")
+					(reference "#PWR0129")
 					(unit 1)
 				)
@@
 		(in_pos_files yes)
 		(dnp no)
-		(property "Reference" "#PWR0118"
+		(property "Reference" "#PWR0131"
 			(at 156.21 106.68 0)
 			(hide yes)
@@
 			(project "LoRa-Monitor"
 				(path "/7510cc7d-c141-46d4-8947-7def3af8cf35/004b7f1f-ea7b-4526-8ebc-4e4b164bf3f3"
-					(reference "#PWR0118")
+					(reference "#PWR0131")
 					(unit 1)
 				)
@@
 		(dnp no)
 		(fields_autoplaced yes)
-		(property "Reference" "U15"
+		(property "Reference" "U14"
 			(at 137.16 66.04 0)
 			(show_name no)
@@
 			(project "LoRa-Monitor"
 				(path "/7510cc7d-c141-46d4-8947-7def3af8cf35/004b7f1f-ea7b-4526-8ebc-4e4b164bf3f3"
-					(reference "U15")
+					(reference "U14")
 					(unit 1)
 				)
@@
 		(in_pos_files yes)
 		(dnp yes)
-		(property "Reference" "C51"
+		(property "Reference" "C58"
 			(at 141.478 123.952 0)
 			(show_name no)
@@
 			(project "LoRa-Monitor"
 				(path "/7510cc7d-c141-46d4-8947-7def3af8cf35/004b7f1f-ea7b-4526-8ebc-4e4b164bf3f3"
-					(reference "C51")
+					(reference "C58")
 					(unit 1)
 				)
@@
 		(dnp no)
 		(fields_autoplaced yes)
-		(property "Reference" "R95"
+		(property "Reference" "R117"
 			(at 96.52 67.3099 0)
 			(show_name no)
@@
 			(project "LoRa-Monitor"
 				(path "/7510cc7d-c141-46d4-8947-7def3af8cf35/004b7f1f-ea7b-4526-8ebc-4e4b164bf3f3"
-					(reference "R95")
+					(reference "R117")
 					(unit 1)
 				)
@@
 		(in_pos_files yes)
 		(dnp no)
-		(property "Reference" "#PWR0120"
+		(property "Reference" "#PWR0128"
 			(at 93.98 90.17 0)
 			(hide yes)
@@
 			(project "LoRa-Monitor"
 				(path "/7510cc7d-c141-46d4-8947-7def3af8cf35/004b7f1f-ea7b-4526-8ebc-4e4b164bf3f3"
-					(reference "#PWR0120")
+					(reference "#PWR0128")
 					(unit 1)
 				)
@@
 		(in_pos_files yes)
 		(dnp no)
-		(property "Reference" "#PWR0119"
+		(property "Reference" "#PWR0127"
 			(at 93.98 67.31 0)
 			(hide yes)
@@
 			(project "LoRa-Monitor"
 				(path "/7510cc7d-c141-46d4-8947-7def3af8cf35/004b7f1f-ea7b-4526-8ebc-4e4b164bf3f3"
-					(reference "#PWR0119")
+					(reference "#PWR0127")
 					(unit 1)
 				)
@@
 		(in_pos_files yes)
 		(dnp yes)
-		(property "Reference" "C50"
+		(property "Reference" "C57"
 			(at 131.318 123.952 0)
 			(show_name no)
@@
 			(project "LoRa-Monitor"
 				(path "/7510cc7d-c141-46d4-8947-7def3af8cf35/004b7f1f-ea7b-4526-8ebc-4e4b164bf3f3"
-					(reference "C50")
+					(reference "C57")
 					(unit 1)
 				)
@@
 		(in_pos_files yes)
 		(dnp no)
-		(property "Reference" "#PWR0128"
+		(property "Reference" "#PWR0126"
 			(at 85.09 82.55 0)
 			(hide yes)
@@
 			(project "LoRa-Monitor"
 				(path "/7510cc7d-c141-46d4-8947-7def3af8cf35/004b7f1f-ea7b-4526-8ebc-4e4b164bf3f3"
-					(reference "#PWR0128")
+					(reference "#PWR0126")
 					(unit 1)
 				)
@@
 		(in_pos_files yes)
 		(dnp no)
-		(property "Reference" "C49"
+		(property "Reference" "C60"
 			(at 175.514 69.088 0)
 			(show_name no)
@@
 			(project "LoRa-Monitor"
 				(path "/7510cc7d-c141-46d4-8947-7def3af8cf35/004b7f1f-ea7b-4526-8ebc-4e4b164bf3f3"
-					(reference "C49")
+					(reference "C60")
 					(unit 1)
 				)
@@
 		(in_pos_files yes)
 		(dnp no)
-		(property "Reference" "C48"
+		(property "Reference" "C59"
 			(at 165.608 69.342 0)
 			(show_name no)
@@
 			(project "LoRa-Monitor"
 				(path "/7510cc7d-c141-46d4-8947-7def3af8cf35/004b7f1f-ea7b-4526-8ebc-4e4b164bf3f3"
-					(reference "C48")
+					(reference "C59")
 					(unit 1)
 				)
@@
 		(in_pos_files yes)
 		(dnp no)
-		(property "Reference" "#PWR0117"
+		(property "Reference" "#PWR0135"
 			(at 210.82 87.63 0)
 			(hide yes)
@@
 			(project "LoRa-Monitor"
 				(path "/7510cc7d-c141-46d4-8947-7def3af8cf35/004b7f1f-ea7b-4526-8ebc-4e4b164bf3f3"
-					(reference "#PWR0117")
+					(reference "#PWR0135")
 					(unit 1)
 				)
@@
 		(dnp yes)
 		(fields_autoplaced yes)
-		(property "Reference" "R100"
+		(property "Reference" "R119"
 			(at 133.35 113.03 90)
 			(show_name no)
@@
 			(project "LoRa-Monitor"
 				(path "/7510cc7d-c141-46d4-8947-7def3af8cf35/004b7f1f-ea7b-4526-8ebc-4e4b164bf3f3"
-					(reference "R100")
+					(reference "R119")
 					(unit 1)
 				)
@@
 		(in_pos_files yes)
 		(dnp no)
-		(property "Reference" "#PWR0121"
+		(property "Reference" "#PWR0132"
 			(at 162.56 67.31 0)
 			(hide yes)
@@
 			(project "LoRa-Monitor"
 				(path "/7510cc7d-c141-46d4-8947-7def3af8cf35/004b7f1f-ea7b-4526-8ebc-4e4b164bf3f3"
-					(reference "#PWR0121")
+					(reference "#PWR0132")
 					(unit 1)
 				)
@@
 		(dnp no)
 		(fields_autoplaced yes)
-		(property "Reference" "R98"
+		(property "Reference" "R116"
 			(at 87.63 82.5499 0)
 			(show_name no)
@@
 			(project "LoRa-Monitor"
 				(path "/7510cc7d-c141-46d4-8947-7def3af8cf35/004b7f1f-ea7b-4526-8ebc-4e4b164bf3f3"
-					(reference "R98")
+					(reference "R116")
 					(unit 1)
 				)
@@
 		(dnp yes)
 		(fields_autoplaced yes)
-		(property "Reference" "R99"
+		(property "Reference" "R118"
 			(at 123.19 113.03 90)
 			(show_name no)
@@
 			(project "LoRa-Monitor"
 				(path "/7510cc7d-c141-46d4-8947-7def3af8cf35/004b7f1f-ea7b-4526-8ebc-4e4b164bf3f3"
-					(reference "R99")
+					(reference "R118")
 					(unit 1)
 				)
@@
 		(in_pos_files yes)
 		(dnp no)
-		(property "Reference" "#PWR0131"
+		(property "Reference" "#PWR0130"
 			(at 138.43 135.89 0)
 			(hide yes)
@@
 			(project "LoRa-Monitor"
 				(path "/7510cc7d-c141-46d4-8947-7def3af8cf35/004b7f1f-ea7b-4526-8ebc-4e4b164bf3f3"
-					(reference "#PWR0131")
+					(reference "#PWR0130")
 					(unit 1)
 				)
@@
 		(in_pos_files yes)
 		(dnp no)
-		(property "Reference" "#PWR0116"
+		(property "Reference" "#PWR0134"
 			(at 210.82 80.01 0)
 			(hide yes)
@@
 			(project "LoRa-Monitor"
 				(path "/7510cc7d-c141-46d4-8947-7def3af8cf35/004b7f1f-ea7b-4526-8ebc-4e4b164bf3f3"
-					(reference "#PWR0116")
+					(reference "#PWR0134")
 					(unit 1)
 				)
@@
 		(in_pos_files yes)
 		(dnp no)
-		(property "Reference" "#PWR0129"
+		(property "Reference" "#PWR0133"
 			(at 172.72 82.55 0)
 			(hide yes)
@@
 			(project "LoRa-Monitor"
 				(path "/7510cc7d-c141-46d4-8947-7def3af8cf35/004b7f1f-ea7b-4526-8ebc-4e4b164bf3f3"
-					(reference "#PWR0129")
+					(reference "#PWR0133")
 					(unit 1)
 				)
